Commit message: changed name to color detector

File: my_robot_description/urdf/common_properties.xacro (robot description, xacro)
@@ -12,4 +12,7 @@
     <material name="red">
         <color rgba="0.75 0 0 1" />
+    </material>
+    <material name="black">
+        <color rgba="0 0 0 1" />
     </material>
     <xacro:macro name="box_inertia" params="m x y z o_xyz o_rpy">
